File: V1/kicad/KeyMatrix.kicad_sch (KiCad schematic)
At the start: 60 parts

Commit message: worked on kicad
Parts:
- renumbered D_R1-C1 to D_C1-R1, D_R2-C1 to D_C1-R2, D_R3-C1 to D_C1-R3, D_R4-C1 to D_C1-R4, D_R5-C1 to D_C1-R5, D_R1-C2 to D_C2-R1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
Other:
- company: (none) -> Thomas Atkins
- title: (none) -> Raven Keyboard
