File: V1/kicad/Raven_Keyboard.kicad_pcb (KiCad board)
At the start: 2 copper layers, 149.9 x 149.9 mm, 117 parts, among them J1 USB_C_2-LAYER_PADS, J12 SPI, J13 CONN_1, J14 I2C, J2 JTAG, J4 JST_2MM_MALE, J7 CONN_021X02, J9 CONN_01, U2 MCP73831, U3 3.3V, U4 AP7361C-33E, U5 AP7361C-33

Commit message: worked on kicad
Parts:
- removed 3V3_LED1, VIN_LED1: JUMPER-SMT_2_NC_TRACE_SILK, MicroMod-Datalogging-CarrierBoard:SMT-JUMPER_2_NC_TRACE_SILK
- removed BYP1: JUMPER-SMT_2_NO_SILK, MicroMod-Datalogging-CarrierBoard:SMT-JUMPER_2_NO_SILK
- removed C8: 1.0uF, MicroMod-Datalogging-CarrierBoard:0603
- removed D5: RED, MicroMod-Datalogging-CarrierBoard:LED-0603
- removed D7: Yellow, MicroMod-Datalogging-CarrierBoard:LED-0603
- removed D_R1-C1, D_R1-C2, D_R1-C3, D_R1-C4, D_R1-C5, D_R1-C6, D_R2-C1, D_R2-C2, D_R2-C3, D_R2-C4, D_R2-C5, D_R2-C6, D_R3-C1, D_R3-C2, D_R3-C3, D_R3-C4, D_R3-C5, D_R3-C6, D_R4-C1, D_R4-C2, D_R4-C3, D_R4-C4, D_R4-C5, D_R4-C6, D_R5-C1, D_R5-C2, D_R5-C3, D_R5-C4, D_R5-C5, D_R5-C6: 1N4148W, Diode_SMD:D_SOD-123
- removed FD1, FD2, FD3, FD4: FIDUCIALUFIDUCIAL, MicroMod-Datalogging-CarrierBoard:FIDUCIAL-MICRO
- removed FRAME1: FRAME-LEDGER, MicroMod-Datalogging-CarrierBoard:CREATIVE_COMMONS
- removed H1, H2, H3, H4: STAND-OFF, MicroMod-Datalogging-CarrierBoard:STAND-OFF
- removed J13: CONN_1, MicroMod-Datalogging-CarrierBoard:1X01_NO_SILK
- removed J14: I2C, MicroMod-Datalogging-CarrierBoard:1X04_NO_SILK
- removed J9: CONN_01, MicroMod-Datalogging-CarrierBoard:1X01_NO_SILK
- removed LOGO3: OSHW-LOGOMINI, MicroMod-Datalogging-CarrierBoard:OSHW-LOGO-MINI
- removed MEAS1: JUMPER, MicroMod-Datalogging-CarrierBoard:COMBO-JUMPER_2_NC_TRACE
- removed MEAS_BATT1: JMP, MicroMod-Datalogging-CarrierBoard:COMBO-JUMPER_2_NC_TRACE
- removed R11: 1k, MicroMod-Datalogging-CarrierBoard:0603
- removed R12: 4.7k, MicroMod-Datalogging-CarrierBoard:0603
- removed R14: 100k, MicroMod-Datalogging-CarrierBoard:0603
- removed SW_R1-C1, SW_R1-C2, SW_R1-C3, SW_R1-C4, SW_R1-C5, SW_R1-C6, SW_R2-C1, SW_R2-C2, SW_R2-C3, SW_R2-C4, SW_R2-C5, SW_R2-C6, SW_R3-C1, SW_R3-C2, SW_R3-C3, SW_R3-C4, SW_R3-C5, SW_R3-C6, SW_R4-C1, SW_R4-C2, SW_R4-C3, SW_R4-C4, SW_R4-C5, SW_R4-C6, SW_R5-C1, SW_R5-C2, SW_R5-C3, SW_R5-C4, SW_R5-C5, SW_R5-C6: , Switch_Keyboard_Kailh:SW_Kailh_Choc_V1_1.00u
- removed U3: 3.3V, MicroMod-Datalogging-CarrierBoard:SOT23-5
- removed U4: AP7361C-33E, Package_TO_SOT_SMD:SOT-223-3_TabPin2
- removed U5: AP7361C-33, MicroMod-Datalogging-CarrierBoard:UDFN-8
- removed VE1: JMP_2, MicroMod-Datalogging-CarrierBoard:SMT-JUMPER_2_NO_SILK
- added 3.3V_Out1: 3.3V Out, MicroMod-Datalogging-CarrierBoard:COMBO-JUMPER_2_NC_TRACE, F.Cu at (162.3, 62.2)
- added D_C1-R1: 1N4148W, Diode_SMD:D_SOD-123, B.Cu at (46.1, 50.8)
- added D_C1-R2: 1N4148W, Diode_SMD:D_SOD-123, B.Cu at (46.1, 68.6)
- added D_C1-R3: 1N4148W, Diode_SMD:D_SOD-123, B.Cu at (46.1, 86.4)
- added D_C1-R4: 1N4148W, Diode_SMD:D_SOD-123, B.Cu at (47.0, 104.1)
- added D_C1-R5: 1N4148W, Diode_SMD:D_SOD-123, B.Cu at (47.0, 123.2)
- added D_C2-R1: 1N4148W, Diode_SMD:D_SOD-123, B.Cu at (64.8, 48.3)
- added D_C2-R2: 1N4148W, Diode_SMD:D_SOD-123, B.Cu at (64.4, 66.0)
- added D_C2-R3: 1N4148W, Diode_SMD:D_SOD-123, B.Cu at (64.8, 83.8)
- added D_C2-R4: 1N4148W, Diode_SMD:D_SOD-123, B.Cu at (64.8, 101.6)
- added D_C2-R5: 1N4148W, Diode_SMD:D_SOD-123, B.Cu at (64.8, 120.7)
- added D_C3-R1: 1N4148W, Diode_SMD:D_SOD-123, B.Cu at (83.8, 45.7)
- added D_C3-R2: 1N4148W, Diode_SMD:D_SOD-123, B.Cu at (83.8, 63.5)
- added D_C3-R3: 1N4148W, Diode_SMD:D_SOD-123, B.Cu at (83.8, 81.3)
- added D_C3-R4: 1N4148W, Diode_SMD:D_SOD-123, B.Cu at (83.4, 99.1)
- added D_C3-R5: 1N4148W, Diode_SMD:D_SOD-123, B.Cu at (84.7, 118.1)
- added D_C4-R1: 1N4148W, Diode_SMD:D_SOD-123, B.Cu at (103.8, 43.2)
- added D_C4-R2: 1N4148W, Diode_SMD:D_SOD-123, B.Cu at (101.6, 58.4)
- added D_C4-R3: 1N4148W, Diode_SMD:D_SOD-123, B.Cu at (102.9, 76.2)
- added D_C4-R4: 1N4148W, Diode_SMD:D_SOD-123, B.Cu at (102.9, 94.0)
- added D_C4-R5: 1N4148W, Diode_SMD:D_SOD-123, B.Cu at (102.9, 115.6)
- added D_C5-R1: 1N4148W, Diode_SMD:D_SOD-123, B.Cu at (121.9, 45.7)
- added D_C5-R2: 1N4148W, Diode_SMD:D_SOD-123, B.Cu at (120.7, 63.5)
- added D_C5-R3: 1N4148W, Diode_SMD:D_SOD-123, B.Cu at (121.9, 81.3)
- added D_C5-R4: 1N4148W, Diode_SMD:D_SOD-123, B.Cu at (121.9, 99.1)
- added D_C5-R5: 1N4148W, Diode_SMD:D_SOD-123, B.Cu at (121.5, 118.1)
- added D_C6-R1: 1N4148W, Diode_SMD:D_SOD-123, B.Cu at (140.6, 48.3)
- added D_C6-R2: 1N4148W, Diode_SMD:D_SOD-123, B.Cu at (141.0, 66.0)
- added D_C6-R3: 1N4148W, Diode_SMD:D_SOD-123, B.Cu at (141.0, 83.8)
- added D_C6-R4: 1N4148W, Diode_SMD:D_SOD-123, B.Cu at (141.0, 101.6)
- added D_C6-R5: 1N4148W, Diode_SMD:D_SOD-123, B.Cu at (141.3, 120.7)
- added IC1: AP7361C-33SP-13, SamacSys_Parts:SOIC127P600X163-9N, F.Cu at (171.4, 66.0)
- added SW_C1-R1: , Switch_Keyboard_Kailh:SW_Kailh_Choc_V1_1.00u, F.Cu at (44.8, 45.7)
- added SW_C1-R2: , Switch_Keyboard_Kailh:SW_Kailh_Choc_V1_1.00u, F.Cu at (44.8, 63.5)
- added SW_C1-R3: , Switch_Keyboard_Kailh:SW_Kailh_Choc_V1_1.00u, F.Cu at (44.8, 81.3)
- added SW_C1-R4: , Switch_Keyboard_Kailh:SW_Kailh_Choc_V1_1.00u, F.Cu at (44.8, 99.1)
- added SW_C1-R5: , Switch_Keyboard_Kailh:SW_Kailh_Choc_V1_1.00u, F.Cu at (44.8, 118.1)
- added SW_C2-R1: , Switch_Keyboard_Kailh:SW_Kailh_Choc_V1_1.00u, F.Cu at (63.5, 43.2)
- added SW_C2-R2: , Switch_Keyboard_Kailh:SW_Kailh_Choc_V1_1.00u, F.Cu at (63.5, 61.0)
- added SW_C2-R3: , Switch_Keyboard_Kailh:SW_Kailh_Choc_V1_1.00u, F.Cu at (63.5, 78.7)
- added SW_C2-R4: , Switch_Keyboard_Kailh:SW_Kailh_Choc_V1_1.00u, F.Cu at (63.5, 96.5)
- added SW_C2-R5: , Switch_Keyboard_Kailh:SW_Kailh_Choc_V1_1.00u, F.Cu at (63.5, 115.6)
- added SW_C3-R1: , Switch_Keyboard_Kailh:SW_Kailh_Choc_V1_1.00u, F.Cu at (82.5, 40.6)
- added SW_C3-R2: , Switch_Keyboard_Kailh:SW_Kailh_Choc_V1_1.00u, F.Cu at (82.5, 58.4)
- added SW_C3-R3: , Switch_Keyboard_Kailh:SW_Kailh_Choc_V1_1.00u, F.Cu at (82.5, 76.2)
- added SW_C3-R4: , Switch_Keyboard_Kailh:SW_Kailh_Choc_V1_1.00u, F.Cu at (82.5, 94.0)
- added SW_C3-R5: , Switch_Keyboard_Kailh:SW_Kailh_Choc_V1_1.00u, F.Cu at (82.5, 113.0)
- added SW_C4-R1: , Switch_Keyboard_Kailh:SW_Kailh_Choc_V1_1.00u, F.Cu at (101.6, 38.1)
- added SW_C4-R2: , Switch_Keyboard_Kailh:SW_Kailh_Choc_V1_1.00u, F.Cu at (101.6, 53.3)
- added SW_C4-R3: , Switch_Keyboard_Kailh:SW_Kailh_Choc_V1_1.00u, F.Cu at (101.6, 71.1)
- added SW_C4-R4: , Switch_Keyboard_Kailh:SW_Kailh_Choc_V1_1.00u, F.Cu at (101.6, 88.9)
- added SW_C4-R5: , Switch_Keyboard_Kailh:SW_Kailh_Choc_V1_1.00u, F.Cu at (101.6, 110.5)
- added SW_C5-R1: , Switch_Keyboard_Kailh:SW_Kailh_Choc_V1_1.00u, F.Cu at (120.7, 40.6)
- added SW_C5-R2: , Switch_Keyboard_Kailh:SW_Kailh_Choc_V1_1.00u, F.Cu at (120.7, 58.4)
- added SW_C5-R3: , Switch_Keyboard_Kailh:SW_Kailh_Choc_V1_1.00u, F.Cu at (120.7, 76.2)
- added SW_C5-R4: , Switch_Keyboard_Kailh:SW_Kailh_Choc_V1_1.00u, F.Cu at (120.7, 94.0)
- added SW_C5-R5: , Switch_Keyboard_Kailh:SW_Kailh_Choc_V1_1.00u, F.Cu at (120.7, 113.0)
- added SW_C6-R1: , Switch_Keyboard_Kailh:SW_Kailh_Choc_V1_1.00u, F.Cu at (139.7, 43.2)
- added SW_C6-R2: , Switch_Keyboard_Kailh:SW_Kailh_Choc_V1_1.00u, F.Cu at (139.7, 61.0)
- added SW_C6-R3: , Switch_Keyboard_Kailh:SW_Kailh_Choc_V1_1.00u, F.Cu at (139.7, 78.7)
- added SW_C6-R4: , Switch_Keyboard_Kailh:SW_Kailh_Choc_V1_1.00u, F.Cu at (139.7, 96.5)
- added SW_C6-R5: , Switch_Keyboard_Kailh:SW_Kailh_Choc_V1_1.00u, F.Cu at (139.7, 115.6)
- C1, C13, C5, C6, C7: footprint MicroMod-Datalogging-CarrierBoard:0603 -> Capacitor_SMD:C_1206_3216Metric_Pad1.33x1.80mm_HandSolder
- D1: footprint MicroMod-Datalogging-CarrierBoard:SOD-323 -> Diode_SMD:D_1206_3216Metric_Pad1.42x1.75mm_HandSolder
- R5: footprint MicroMod-Datalogging-CarrierBoard:0603 -> Resistor_SMD:R_1206_3216Metric_Pad1.30x1.75mm_HandSolder
- moved R6 206.8 mm to (198.1, 35.6), turned to 180 degrees
- moved J7 193.6 mm to (203.2, 50.8)
- moved U2 188.3 mm to (195.6, 40.6)
- moved J4 186.8 mm to (206.9, 41.9), turned to -90 degrees
- moved C4 186.4 mm to (191.8, 54.6)
- moved C3 183.0 mm to (195.6, 48.3), turned to 180 degrees
- moved D2 174.3 mm to (190.5, 35.6), turned to 180 degrees
- moved R7 173.1 mm to (190.5, 40.6), turned to 180 degrees
- moved D3 171.5 mm to (196.8, 58.4)
- moved S1 166.2 mm to (193.0, 91.4)
- moved C13 163.1 mm to (179.1, 72.4)
- moved C1 161.0 mm to (179.1, 68.6)
- moved S2 152.6 mm to (193.0, 104.1)
- moved C6 151.3 mm to (162.3, 71.1), turned to 180 degrees
- moved C5 148.9 mm to (162.3, 67.3), turned to 180 degrees
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Connections:
- C1 pad 1: VIN -> 5V
- C13 pad 1: VIN -> 5V
- C2 pad +: VIN -> 5V
- F2 pad 2: VIN -> 5V
- MicroMod_Connector1 pad 72: /RTC_3V -> unconnected-(MicroMod_Connector1-Pad72)
- MicroMod_Connector1 pad 9: VIN -> 5V
- R10 pad 2: VIN -> 5V
- R5 pad 1: Net-(D1-PadC) -> 5V
- R5 pad 2: VIN -> /3.3V_EN
Routing:
- net Row_3: track 0.00 -> 106.6 mm
- net Row_2: track 0.00 -> 105.2 mm
- net Row_4: track 0.00 -> 104.3 mm
- net Row_1: track 0.00 -> 101.9 mm
- net Row_5: track 0.00 -> 101.1 mm
- net Col_1: track 0.00 -> 77.7 mm
- net Col_4: track 0.00 -> 77.2 mm
- net Col_6: track 0.00 -> 76.0 mm
- net Col_2: track 0.00 -> 76.0 mm
- net Col_5: track 21.0 -> 76.0 mm
- net Col_3: track 21.9 -> 76.0 mm
- net Net-(D_R1-C3-Pad2): track 44.1 -> 0.00 mm
- net Net-(D_C3-R5-Pad2): track 0.00 -> 16.1 mm
- net Net-(D_C6-R5-Pad2): track 0.00 -> 13.1 mm
- net Net-(D_C2-R2-Pad2): track 0.00 -> 12.9 mm
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Other:
- board outline removed
