File: V1/kicad/Raven_Keyboard.kicad_sch (KiCad schematic)
At the start: 57 parts, among them J1 USB_C_2-LAYER_PADS, J12 SPI, J13 CONN_1, J14 I2C, J2 JTAG, J4 JST_2MM_MALE, J7 CONN_021X02, J9 CONN_01, U2 MCP73831, U3 3.3V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

Commit message: worked on kicad
Parts:
- removed 3V3_LED1, VIN_LED1: JUMPER-SMT_2_NC_TRACE_SILK, SMT-JUMPER_2_NC_TRACE_SILK, symbol MicroMod-Datalogging-CarrierBoard-eagle-import:JUMPER-SMT_2_NC_TRACE_SILK
- removed BYP1: JUMPER-SMT_2_NO_SILK, SMT-JUMPER_2_NO_SILK, symbol MicroMod-Datalogging-CarrierBoard-eagle-import:JUMPER-SMT_2_NO_SILK
- removed C8: 1.0uF, 0603, symbol MicroMod-Datalogging-CarrierBoard-eagle-import:1.0UF-0603-16V-10%
- removed D1: 3.3V, SOD-323, symbol MicroMod-Datalogging-CarrierBoard-eagle-import:DIODE-ZENER-MM3Z3V3T1G
- removed D5: RED, LED-0603, symbol MicroMod-Datalogging-CarrierBoard-eagle-import:LED-RED0603
- removed D7: Yellow, LED-0603, symbol MicroMod-Datalogging-CarrierBoard-eagle-import:LED-YELLOW0603
- removed FD1, FD2, FD3, FD4: FIDUCIALUFIDUCIAL, FIDUCIAL-MICRO, symbol MicroMod-Datalogging-CarrierBoard-eagle-import:FIDUCIALUFIDUCIAL
- removed FRAME1: FRAME-LEDGER, CREATIVE_COMMONS, symbol MicroMod-Datalogging-CarrierBoard-eagle-import:FRAME-LEDGER
- removed H1, H2, H3, H4: STAND-OFF, STAND-OFF, symbol MicroMod-Datalogging-CarrierBoard-eagle-import:STAND-OFF
- removed J13: CONN_1, 1X01_NO_SILK, symbol MicroMod-Datalogging-CarrierBoard-eagle-import:CONN_01PTH_NO_SILK_YES_STOP
- removed J14: I2C, 1X04_NO_SILK, symbol MicroMod-Datalogging-CarrierBoard-eagle-import:I2C_STANDARD_NO_SILK
- removed J9: CONN_01, 1X01_NO_SILK, symbol MicroMod-Datalogging-CarrierBoard-eagle-import:CONN_01PTH_NO_SILK_YES_STOP
- removed LOGO3: OSHW-LOGOMINI, OSHW-LOGO-MINI, symbol MicroMod-Datalogging-CarrierBoard-eagle-import:OSHW-LOGOMINI
- removed MEAS_BATT1: JMP, COMBO-JUMPER_2_NC_TRACE, symbol MicroMod-Datalogging-CarrierBoard-eagle-import:JUMPER-COMBO_2_NC_TRACE
- removed R11: 1k, 0603, symbol MicroMod-Datalogging-CarrierBoard-eagle-import:1KOHM-0603-1/10W-1%
- removed R12: 4.7k, 0603, symbol MicroMod-Datalogging-CarrierBoard-eagle-import:4.7KOHM-0603-1/10W-1%
- removed R14, R5: 100k, 0603, symbol MicroMod-Datalogging-CarrierBoard-eagle-import:100KOHM-0603-1/10W-1%
- removed U3: 3.3V, SOT23-5, symbol MicroMod-Datalogging-CarrierBoard-eagle-import:V_REG_AP2112K-3.3V
- removed U4: AP7361C-33E, Package_TO_SOT_SMD:SOT-223-3_TabPin2, symbol Regulator_Linear:AP7361C-33E
- removed U5: AP7361C-33, UDFN-8, symbol MicroMod-Datalogging-CarrierBoard-eagle-import:AP7361C-33FGEUDFN-8
- removed VE1: JMP_2, SMT-JUMPER_2_NO_SILK, symbol MicroMod-Datalogging-CarrierBoard-eagle-import:JUMPER-SMT_2_NO_SILK
- added D1: 3.3V, Diode_SMD:D_1206_3216Metric_Pad1.42x1.75mm_HandSolder, symbol Device:D_Zener_Small_Filled
- added IC1: AP7361C-33SP-13, SOIC127P600X163-9N, symbol SamacSys_Parts:AP7361C-33SP-13
- added R5: 100k, Resistor_SMD:R_1206_3216Metric_Pad1.30x1.75mm_HandSolder, symbol Device:R_Small
- 3.3V_Out1: renamed from MEAS1; value JUMPER -> 3.3V Out
- C1, C13, C5, C6, C7: footprint 0603 -> Capacitor_SMD:C_1206_3216Metric_Pad1.33x1.80mm_HandSolder
- R6: symbol MicroMod-Datalogging-CarrierBoard-eagle-import:2.2KOHM-0603-1/10W-1% -> Device:R
Connections:
- net VIN is gone; now on net 5V: C1.1, C13.1, C2.+, F2.2, MicroMod_Connector1.9 (USB_VIN), R10.2
- net 3.3V: now also 3.3V_Out1.1, 3.3V_Out1.3 (1); no longer 3.3V_Out1.2, 3.3V_Out1.4 (2)
- net 3.3V_EN: now also D1.1 (K), IC1.2 (EN), R5.2
- net 5V: now also IC1.8 (IN), R5.1
- net GND: now also D1.2 (A), IC1.4 (GND)
- net RTC_3V: no longer names the net of MicroMod_Connector1.72 (RTC_3V)
- new net: 3.3V_Out1.2, 3.3V_Out1.4 (2), IC1.1 (OUT)
- new net: IC1.3 (NC_1), IC1.5 (NC_2), IC1.6 (NC_3), IC1.7 (NC_4)
Other:
- note added: "Buttons"
- note added: "SWD"
- note removed: "Close VE to enable processor control of 3.3V bus."
- note removed: "Closing jumper bypasses PTC to allow >2A current flows."
- note removed: "Peripheral Power Control"
- note removed: "SWO"
- note removed: "VIN: 3.7-6.0V"
- company: (none) -> Thomas Atkins
- title: (none) -> Raven Keyboard
- moved on the sheet: 3.3V_Out1, C1, C13, C2, C3, C4, C5, C6, C7, D2, D3, H5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
